Commit message: P2 D7: line-following track world + camera chain
赛道：scripts/make_line_world.py 参数化生成 worlds/line_following.world
（9.42 m 环线、28 段 FlatBlack 薄盒、视觉-only 无 collision 以免污染 /odom）。

相机：挂点从车壳内 (0.18,0,0.045) 移到车壳外 (0.21,0,0.055)，离地 0.154 m；
camera_pitch 抽成 xacro arg（默认 0 保持 D5 口径），巡线取 +0.6 rad
——URDF 绕 y 正角才是低头，写成 -0.6 会抬头拍到天空背景色（std=0 的纯色图）。

慢仿真对策：cmd_vel_timeout 按仿真时间计时，RTF 0.11~0.22 下 0.5 s 会被
DDS 成簇投递打穿，表现为车每隔几秒自顿（10→200 Hz 提频无效）。新增
config/mybot_controllers_slowsim.yaml 作为第二个 <parameters> 标签覆盖为 5.0 s，
真机仍回 0.5 s。

验证脚本：snap_camera.py（抓帧 + 逐行线中心统计，起点 6 行全命中、
横向偏差 -0.01）、drive_check.py（按仿真时间开车打表，0.2 m/s 连续 8 s 无掉零）。

File: mybot/urdf/mybot.ros2c.urdf.xacro (robot description, xacro)
@@ -6,4 +6,8 @@
   <xacro:arg name="ros2c_params_file"
              default="$(find mybot_description)/config/mybot_controllers.yaml"/>
+  <!-- D7：第二个参数文件，只用于覆盖个别键（gazebo_ros2_control 读多个 <parameters> 标签，
+       后者覆盖前者）。默认与主文件相同 = 不覆盖，保持 D4 验收口径；
+       巡线 launch 传 config/mybot_controllers_slowsim.yaml 放宽 cmd_vel_timeout。 -->
+  <xacro:arg name="extra_params_file" default="$(arg ros2c_params_file)"/>
   <xacro:include filename="$(find mybot_description)/urdf/mybot_core.urdf.xacro"/>
   <!-- D5: 传感器（激光/相机）与硬件抽象层解耦，两种驱动外壳都 include 同一份 -->
@@ -33,5 +37,8 @@
   <gazebo>
     <plugin name="gazebo_ros2_control" filename="libgazebo_ros2_control.so">
+      <!-- 多个参数文件 = 多个 <parameters> 标签（实测写成空格分隔的单个标签会被当成一个路径，
+           报 "Error opening YAML file"）；后一个标签里的键覆盖前一个 -->
       <parameters>$(arg ros2c_params_file)</parameters>
+      <parameters>$(arg extra_params_file)</parameters>
       <controller_manager_name>controller_manager</controller_manager_name>
       <ros>

File: mybot/urdf/mybot_core.urdf.xacro (robot description, xacro)
@@ -118,8 +118,22 @@
   </joint>
   <link name="camera_link"/>
+  <!-- D7 修正：原挂点 xyz="0.18 0 0.045" 落在车体壳内（底盘半长 0.20、顶面 z=0.03），
+       相机往下看会先撞到自家顶板，巡线时前景全是蓝色车壳。
+       现移到车体外前方：x=0.21（前壁外 1 cm）、z=0.055（顶面上方 2.5 cm），
+       距地高度 = 0.099(底盘中心离地) + 0.055 = 0.154 m。
+       pitch 抽成 arg：默认 0.0 保持 D5 的话题/TF 验收口径不变，
+       巡线 launch 传 +0.6 rad（约 +34°）。**符号注意**：URDF 绕 y 轴正角 = 低头
+       （+x 转向 −z），写成 -0.6 会变成抬头看天，画面就是一张 Gazebo 天空色（178）的纯色图。
+       为什么是 0.6：
+       hfov=1.2 rad、320x240 → vfov/2 = atan(tan(0.6)*240/320) = 0.474 rad，
+       pitch 必须大于 0.474（低头）整幅画面才全部落在地面上；0.6 时
+       最近可见点 0.154/tan(61.5°)=0.084 m、最远 0.154/tan(7.2°)=1.22 m（均在车前） -->
+  <xacro:property name="camera_x" value="0.21"/>
+  <xacro:property name="camera_z" value="0.055"/>
+  <xacro:arg name="camera_pitch" default="0.0"/>
   <joint name="camera_joint" type="fixed">
     <parent link="base_link"/>
     <child link="camera_link"/>
-    <origin xyz="0.18 0 0.045" rpy="0 0 0"/>
+    <origin xyz="${camera_x} 0 ${camera_z}" rpy="0 $(arg camera_pitch) 0"/>
   </joint>
   <!-- ============ Gazebo 物理与差速驱动插件（D3） ============ -->
